File: schematics/Generic_Front_Panel/Generic_Front_Panel.kicad_pcb (KiCad board)
At the start: 2 copper layers, 194.9 x 90.2 mm, 74 parts, among them J1 Interface, SW1 Reset, SW10 D, SW11 CMD2, SW12 2, SW13 6, SW14 A, SW15 E, SW16 CMD3, SW17 3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

Commit message: Update filter capacitor to 100uF
Parts:
- C12: value 47uF -> 100uF
Changed lines of the file:
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@@
 			)
 		)
-		(property "Value" "47uF"
+		(property "Value" "100uF"
 			(at 1.25 -4.4 0)
 			(layer "B.Fab")
